File: WaterCam_mDot_WittyPi_AHT_BNO_Lepton.kicad_sch (KiCad schematic)
At the start: 8 parts, among them J1 GPIO, J2 FLIR Lepton Socket, J3 Witty Pi 4 L3V7 P3 Header, Q1 NMOS, U1 ATH20, U2 BNO055(IMU), U3 MDOT

Commit message: Correct schematic wiring and add missing components for WaterCam HAT
Fixes applied to WaterCam_mDot_WittyPi_AHT_BNO_Lepton.kicad_sch to match
the SU-WaterCam software wiring and Raspberry Pi HAT specification.

Fix 1 — mDot UART5 wiring:
- mDot PA_2 (TX) → GPIO13/RXD5 (UART5 RX), Pi pin 33
- mDot PA_3 (RX) → GPIO12/TXD5 (UART5 TX), Pi pin 32
- Uses /dev/ttyAMA5, dtoverlay=uart5

Fix 2 — GPIO17 conflict resolved:
- Removed erroneous bridge from J2-P15 to GPIO17 (WittyPi-reserved pin)
- J2-P15 (Lepton VSYNC/GPIO2) now correctly routed to GPIO24 (Pi pin 18)

Fix 3 — Lepton Breakout Board v2 J2 connector pinout:
- P1: SDA (I2C CCI), P3: SPI CLK, P5: SPI MOSI, P8: SPI CS
- P12: SPI MISO, P15: GPIO24 (VSYNC), P17: GPIO6 (RESET_L), P19: SCL
- Remaining pins: +5V (P2), no_connect, or GND as per breakout board spec

Fix 4 — mDot VDD power source corrected to WittyPi always-on 3.3V:
- mDot powered from J3-3V3 (WittyPi internal MCU/RTC supply, always-on)
- NOT from Pi +3V3, which is cut entirely when WittyPi shuts the Pi down
- 6-wire chain: mDot VDD → (179.07,83.82) → J3 pin 2 (231.14,35.56)

Fix 5 — Lepton PW_DWN_L (J2-P18):
- Changed from no_connect to +3V3 (always-on, Lepton never powered down)

Fix 6 — I2C pull-up resistors (R6, R7):
- R6 4.7kΩ on GPIO2/SDA1, R7 4.7kΩ on GPIO3/SCL1
- Covers AHT20, BNO055/085, and Lepton CCI on I2C bus 1

Fix 7 — HAT ID EEPROM (U4, CAT24C256, SOIC-8):
- New CAT24C256 lib symbol defined inline (Memory_EEPROM:CAT24C256)
- Address 0x50: A0/A1/A2/WP all tied to GND; VCC to +3V3
- SDA → ID_SDA net (GPIO0, Pi pin 27); SCL → ID_SCL net (GPIO1, Pi pin 28)
- R4 3.9kΩ pull-up on ID_SDA, R5 3.9kΩ pull-up on ID_SCL (per HAT spec)
- Connects to existing ID_SDA/ID_SCL labels already wired to J1 GPIO0/GPIO1

Fix 8 — Decoupling capacitors (C1–C6):
- C1 100µF + C2 100nF on mDot VDD (bulk + bypass for LoRa TX transients)
- C3 100nF + C4 10µF on AHT20 VDD; C5 100nF on BNO055 VDD
- C6 100nF on Lepton +5V (VIN, J2-P2)

Fix 9 — mDot NRESET pull-up (R9):
- R9 10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
Parts:
- added C1: 100µF, Capacitor_THT:CP_Radial_D5.0mm_P2.00mm, symbol Device:C_Small
- added C2, C3, C5, C6: 100nF, Capacitor_SMD:C_0402_1005Metric, symbol Device:C_Small
- added C4: 10µF, Capacitor_SMD:C_0805_2012Metric, symbol Device:C_Small
- added J4: IR_CUT_Camera, Connector_PinHeader_2.54mm:PinHeader_1x04_P2.54mm_Vertical, symbol Connector_Generic:Conn_01x04
- added R4, R5: 3.9kΩ, Resistor_SMD:R_0402_1005Metric, symbol Device:R_Small
- added R6, R7: 4.7kΩ, Resistor_SMD:R_0402_1005Metric, symbol Device:R_Small
- added R8: 100Ω, Resistor_SMD:R_0402_1005Metric, symbol Device:R_Small
- added R9: 10kΩ, Resistor_SMD:R_0402_1005Metric, symbol Device:R_Small
- added U4: CAT24C256, Package_SO:SOIC-8_3.9x4.9mm_P1.27mm, symbol Memory_EEPROM:CAT24C256
- Q1: value NMOS -> 2N7002; footprint IRLB8721PBF Model:TO254P1067X483X2057-3 -> Package_TO_SOT_SMD:SOT-23
Connections:
- net +5V: now also C6.1
- net GND: now also C1.2, C2.2, C3.2, C4.2, C5.2, C6.2, U4.1 (A0); no longer J2.1 (Pin_1)
- net GPIO10/SPI0.MOSI: now also J2.5 (Pin_5); no longer J2.9 (Pin_9)
- net GPIO11/SPI0.SCLK: now also J2.3 (Pin_3); no longer J2.7 (Pin_7)
- net GPIO17: no longer J2.15 (Pin_15)
- net GPIO22: now also J4.2 (Pin_2)
- net GPIO24: now also J2.15 (Pin_15)
- net GPIO27: now also J4.1 (Pin_1)
- net GPIO2/SDA1: now also J2.1 (Pin_1), R6.2; no longer J2.5 (Pin_5)
- net GPIO3/SCL1: now also J2.19 (Pin_19), R7.2; no longer J2.8 (Pin_8)
- net GPIO8/SPI0.CE0: now also J2.8 (Pin_8); no longer J2.10 (Pin_10)
- net ID_SCL: now also R5.2
- net ID_SDA: now also R4.2
- net at J3.2 (3V3), U3.1 (VDD): now also C1.1, C2.1
- net at R3.2, U3.19 (PB_1): now also R8.1; no longer Q1.2 (G)
- net at U3.5 (NRESET): now also R9.2
- new net: Q1.2 (G), R8.2
- no-connect marks 61 -> 63

Commit message: Fix GPIO17, MASTER_CLK, WittyPi SW short, Q1 mis-pinning; OSHPark rules
Rebased onto main after #1 (schematic corrections). The schematic and board
are this commit's versions: they build on #1's corrections and deliberately
drop U4/R4/R5 (HAT EEPROM not needed; overlays load from config.txt) and J4
(the IR-cut circuit is deferred as external to the HAT), as recorded in
WaterCam_PCB_Design_Changes_Required.md.

Left out of the public repo: KiCad auto-backup zips, autosave/lock/-bak
files, per-user .kicad_prl and .history, and the vendor datasheets and
manuals (References/README.md lists where to get them). .gitignore keeps
them out.

Co-Authored-By: Claude Opus 5.5 <noreply@anthropic.com>
Parts:
- removed J4: IR_CUT_Camera, Connector_PinHeader_2.54mm:PinHeader_1x04_P2.54mm_Vertical, symbol Connector_Generic:Conn_01x04
- removed R4, R5: 3.9kΩ, Resistor_SMD:R_0402_1005Metric, symbol Device:R_Small
- removed U4: CAT24C256, Package_SO:SOIC-8_3.9x4.9mm_P1.27mm, symbol Memory_EEPROM:CAT24C256
- C1: footprint Capacitor_THT:CP_Radial_D5.0mm_P2.00mm -> Capacitor_SMD:C_0805_2012Metric
- C4: footprint Capacitor_SMD:C_0805_2012Metric -> Capacitor_SMD:C_0402_1005Metric
- Q1: value 2N7002 -> BSS138; symbol Simulation_SPICE:NMOS -> Transistor_FET:BSS138
Connections:
- net +5V: now also C3.1, C4.1, C5.1
- net GND: now also J2.1 (Pin_1), Q1.2 (S); no longer Q1.3 (S)
- net GPIO10/SPI0.MOSI: now also J2.9 (Pin_9); no longer J2.5 (Pin_5)
- net GPIO11/SPI0.SCLK: now also J2.7 (Pin_7); no longer J2.3 (Pin_3)
- net GPIO16: now also U2.1 (RST)
- net GPIO20/PCM.DIN: now also U2.10 (INT)
- net GPIO24: no longer J2.15 (Pin_15)
- net GPIO2/SDA1: now also J2.5 (Pin_5); no longer J2.1 (Pin_1)
- net GPIO3/SCL1: now also J2.8 (Pin_8); no longer J2.19 (Pin_19)
- net GPIO8/SPI0.CE0: now also J2.10 (Pin_10); no longer J2.8 (Pin_8)
- net +3V3: now reaches J1.1 (Pin_1)
- net +3V3: now also R6.1, R7.1
- net WP_3V3: now reaches C1.1, C2.1, J3.2 (3V3), U3.1 (VDD)
- net WP_3V3: now also R9.1
- net at Q1.1 (G): now also R8.1; no longer J3.5 (SW)
- net at R3.2, U3.19 (PB_1): now also R8.2; no longer R8.1
- net GPIO17: no longer names the net of J1.11 (Pin_11)
- net ID_SCL: no longer names the net of J1.28 (Pin_28)
- net ID_SDA: no longer names the net of J1.27 (Pin_27)
- new net WP_SW: J3.5 (SW), Q1.3 (D)
- no-connect marks 63 -> 57
Other:
- moved on the sheet: J2, J3, Q1, R3, U3

Commit message: v6 work in progress: BNO055 fixes, sensor rails, placement (not yet routed)
Checkpoint of the 2026-09-09 session on top of the OSHPark-rules commit:
- Schematic: BNO055 fixes, sensor power rails, U2 INT no-connect.
- PCB: F8, component placement and fixes from that session; all 22
  footprints on the board, 0 shorts and 0 solder-mask bridges (were 8/8).
- SESSION_HANDOFF.md: status, the remaining DRC items, routing order,
  open assembly decisions, and two risks to check before ordering (BNO055
  pad 1 has no orientation marking; MDOT footprint duplicates pad 24).

Not orderable: 26 connections unrouted, 17 DRC violations.

tools/kicad_pin_positions.py and tools/pdf_vector_extract.py are the
session's helper scripts turned into small CLI tools (paths are arguments).

Co-Authored-By: Claude Opus 5.5 <noreply@anthropic.com>
Connections:
- net +3V3: now also C3.1, C4.1, C5.1, U1.1 (VIN), U2.6 (VIN)
- net +5V: no longer C3.1, C4.1, C5.1, U1.1 (VIN), U2.6 (VIN)
- net GPIO20/PCM.DIN: no longer U2.10 (INT)
- net GPIO2/SDA1: now also U2.2 (SDA); no longer U2.3 (SCL)
- net GPIO3/SCL1: now also U2.3 (SCL); no longer U2.2 (SDA)
- no-connect marks 57 -> 58
Changed lines of the file:
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@@
 	)
 	(no_connect
+		(at 156.21 35.56)
+	)
+	(no_connect
 		(at 60.96 40.64)
 	)
@@
 	(wire
 		(pts
-			(xy 127 43.18) (xy 138.43 43.18)
+			(xy 127.0 46.99) (xy 138.43 46.99)
 		)
 		(stroke
@@
 	(wire
 		(pts
-			(xy 127 88.9) (xy 127 43.18)
+			(xy 127.0 88.9) (xy 127.0 46.99)
 		)
 		(stroke
@@
 	(wire
 		(pts
-			(xy 129.54 46.99) (xy 138.43 46.99)
+			(xy 129.54 43.18) (xy 138.43 43.18)
 		)
 		(stroke
@@
 	(wire
 		(pts
-			(xy 129.54 46.99) (xy 129.54 90.17)
+			(xy 129.54 43.18) (xy 129.54 90.17)
 		)
 		(stroke
@@
 		)
 	)
-	(label "GPIO20{slash}PCM.DIN"
-		(at 156.21 35.56 0)
-		(effects
-			(font
-				(size 1.27 1.27)
-			)
-			(justify left bottom)
-		)
-	)
 	(label "GPIO16"
 		(at 138.43 50.8 180)
@@
 	)
 	(symbol
-		(lib_id "power:+5V")
+		(lib_id "power:+3V3")
 		(at 40.64 113.03 0)
 		(unit 1)
@@
 			)
 		)
-		(property "Value" "+5V"
+		(property "Value" "+3V3"
 			(at 41.0083 108.7056 0)
 			(show_name no)
@@
 	)
 	(symbol
-		(lib_id "power:+5V")
+		(lib_id "power:+3V3")
 		(at 134.62 29.21 0)
 		(unit 1)
@@
 			)
 		)
-		(property "Value" "+5V"
+		(property "Value" "+3V3"
 			(at 134.9883 24.8856 0)
 			(show_name no)
@@
 	)
 	(symbol
-		(lib_id "power:+5V")
+		(lib_id "power:+3V3")
 		(at 304.8 158.496 0)
 		(unit 1)
@@
 			)
 		)
-		(property "Value" "+5V"
+		(property "Value" "+3V3"
 			(at 305.1683 155.0716 0)
 			(show_name no)
@@
 	)
 	(symbol
-		(lib_id "power:+5V")
+		(lib_id "power:+3V3")
 		(at 312.42 158.496 0)
 		(unit 1)
@@
 			)
 		)
-		(property "Value" "+5V"
+		(property "Value" "+3V3"
 			(at 312.7883 155.0716 0)
 			(show_name no)
@@
 	)
 	(symbol
-		(lib_id "power:+5V")
+		(lib_id "power:+3V3")
 		(at 320.04 158.496 0)
 		(unit 1)
@@
 			)
 		)
-		(property "Value" "+5V"
+		(property "Value" "+3V3"
 			(at 320.4083 155.0716 0)
 			(show_name no)
